File: KiCad/Soney.kicad_sch (KiCad schematic)
At the start: 22 parts, among them J1 12-18VDC, J2 Left, J3 Right, J4 External Input, J5 External Link, SW1 Power, SW2 Driver Select 5A

Commit message: Schematic adjustment
Parts:
- D1: value Red -> Red (Exterior)
Other:
- moved on the sheet: D1, R1
Changed lines of the file:
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@@
 	)
 	(rectangle
-		(start 74.93 63.5)
+		(start 83.82 63.5)
 		(end 170.18 93.98)
 		(stroke
@@
 	)
 	(junction
-		(at 80.01 90.17)
+		(at 76.2 90.17)
 		(diameter 0)
 		(color 0 0 0 0)
 	)
 	(junction
-		(at 80.01 67.31)
+		(at 76.2 67.31)
 		(diameter 0)
 		(color 0 0 0 0)
@@
 	(wire
 		(pts
-			(xy 80.01 76.2) (xy 80.01 77.47)
-		)
-		(stroke
-			(width 0)
-			(type default)
-		)
-	)
-	(wire
-		(pts
-			(xy 80.01 85.09) (xy 80.01 90.17)
+			(xy 76.2 76.2) (xy 76.2 77.47)
+		)
+		(stroke
+			(width 0)
+			(type default)
+		)
+	)
+	(wire
+		(pts
+			(xy 76.2 85.09) (xy 76.2 90.17)
 		)
 		(stroke
@@
 	(wire
 		(pts
-			(xy 80.01 90.17) (xy 90.17 90.17)
+			(xy 76.2 90.17) (xy 90.17 90.17)
 		)
 		(stroke
@@
 	(wire
 		(pts
-			(xy 80.01 67.31) (xy 80.01 71.12)
+			(xy 76.2 67.31) (xy 76.2 71.12)
 		)
 		(stroke
@@
 	(wire
 		(pts
-			(xy 80.01 67.31) (xy 90.17 67.31)
-		)
-		(stroke
-			(width 0)
-			(type default)
-		)
-	)
-	(wire
-		(pts
-			(xy 69.85 67.31) (xy 80.01 67.31)
+			(xy 76.2 67.31) (xy 90.17 67.31)
+		)
+		(stroke
+			(width 0)
+			(type default)
+		)
+	)
+	(wire
+		(pts
+			(xy 69.85 67.31) (xy 76.2 67.31)
 		)
 		(stroke
@@
 	(wire
 		(pts
-			(xy 49.53 90.17) (xy 80.01 90.17)
+			(xy 49.53 90.17) (xy 76.2 90.17)
 		)
 		(stroke
@@
 	(symbol
 		(lib_id "Device:LED")
-		(at 80.01 81.28 90)
+		(at 76.2 81.28 90)
 		(unit 1)
 		(exclude_from_sim no)
@@
 		(on_board yes)
 		(dnp no)
-		(fields_autoplaced yes)
 		(property "Reference" "D1"
-			(at 83.82 81.5974 90)
+			(at 70.866 80.518 90)
 			(effects
 				(font
@@
 			)
 		)
-		(property "Value" "Red"
-			(at 83.82 84.1374 90)
+		(property "Value" "Red (Exterior)"
+			(at 59.944 83.058 90)
 			(effects
 				(font
@@
 		)
 		(property "Footprint" ""
-			(at 80.01 81.28 0)
+			(at 76.2 81.28 0)
 			(effects
 				(font
@@
 		)
 		(property "Datasheet" "~"
-			(at 80.01 81.28 0)
+			(at 76.2 81.28 0)
 			(effects
 				(font
@@
 		)
 		(property "Description" "Light emitting diode"
-			(at 80.01 81.28 0)
+			(at 76.2 81.28 0)
 			(effects
 				(font
@@
 		)
 		(property "Sim.Pins" "1=K 2=A"
-			(at 80.01 81.28 0)
+			(at 76.2 81.28 0)
 			(effects
 				(font
@@
 	(symbol
 		(lib_id "Device:R_Small_US")
-		(at 80.01 73.66 0)
+		(at 76.2 73.66 0)
 		(unit 1)
 		(exclude_from_sim no)
@@
 		(fields_autoplaced yes)
 		(property "Reference" "R1"
-			(at 82.55 72.3899 0)
+			(at 78.74 72.3899 0)
 			(effects
 				(font
@@
 		)
 		(property "Value" "2K2"
-			(at 82.55 74.9299 0)
+			(at 78.74 74.9299 0)
 			(effects
 				(font
@@
 		)
 		(property "Footprint" ""
-			(at 80.01 73.66 0)
+			(at 76.2 73.66 0)
 			(effects
 				(font
@@
 		)
 		(property "Datasheet" "~"
-			(at 80.01 73.66 0)
+			(at 76.2 73.66 0)
 			(effects
 				(font
@@
 		)
 		(property "Description" "Resistor, small US symbol"
-			(at 80.01 73.66 0)
-			(effects
-				(font
+			(at 76.2 73.66 0)
+			(effects
+				(font
